File: projects/NECTEC/LRTU/communication_module_20190805.brd (EAGLE design)
At the start: 121.1 x 70.6 mm, 47 parts, among them Q1 BC847BS, U1 ESP-WROOM-32U (w/uFL), U2 IMAS980TH, U3 WG209_3E6, U4 RFM95W_SMT, X1 uFL, X2 uFL

Commit message: Revise many things after dealing with Aj.Doy.
Connections:
- net IM_RXD renamed IM_RX
- net IM_TXD renamed IM_TX
- net SCL0_MID/RTC/CAM renamed SCL_MID/RTC/CAM
- net SDA0_MID/RTC/CAM renamed SDA_MID/RTC/CAM
- net SPI1_CE0_1U renamed SPI_CE0_1U
- net SPI1_CE1_1U renamed SPI_CE1_1U
- net SPI1_MISO_1U renamed SPI_MISO_1U
- net SPI1_MOSI_1U renamed SPI_MOSI_1U
- net SPI1_SCLK_1U renamed SPI_SCLK_1U
- removed net NC14: JP11.14
- removed net NC16: JP11.16
Changed lines of the file:
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@@
 <wire x1="110.49" y1="6.35" x2="99.06" y2="22.86" width="0" layer="19" extent="1-1"/>
 </signal>
-<signal name="SPI1_MISO_1U">
+<signal name="SPI_MISO_1U">
 <contactref element="JP11" pad="4"/>
 <contactref element="JP8" pad="3"/>
 <wire x1="-159.2072" y1="-213.36" x2="99.06" y2="25.4" width="0" layer="19" extent="1-1"/>
 </signal>
-<signal name="SPI1_MOSI_1U">
+<signal name="SPI_MOSI_1U">
 <contactref element="JP11" pad="6"/>
 <contactref element="JP6" pad="3"/>
 <wire x1="-138.8872" y1="-213.36" x2="99.06" y2="27.94" width="0" layer="19" extent="1-1"/>
 </signal>
-<signal name="SPI1_CE1_1U">
+<signal name="SPI_CE1_1U">
 <contactref element="JP11" pad="12"/>
 <contactref element="JP5" pad="3"/>
@@
 <wire x1="99.06" y1="45.72" x2="47.858" y2="8.524" width="0" layer="19" extent="1-1"/>
 </signal>
-<signal name="SPI1_CE0_1U">
+<signal name="SPI_CE0_1U">
 <contactref element="JP11" pad="10"/>
 </signal>
-<signal name="SPI1_SCLK_1U">
+<signal name="SPI_SCLK_1U">
 <contactref element="JP11" pad="8"/>
 <contactref element="JP7" pad="3"/>
 <wire x1="-149.0472" y1="-213.36" x2="99.06" y2="30.48" width="0" layer="19" extent="1-1"/>
 </signal>
-<signal name="SCL0_MID/RTC/CAM">
+<signal name="SCL_MID/RTC/CAM">
 <contactref element="JP11" pad="7"/>
 <contactref element="U1" pad="36"/>
 <wire x1="101.6" y1="30.48" x2="47.858" y2="18.684" width="0" layer="19" extent="1-1"/>
 </signal>
-<signal name="SDA0_MID/RTC/CAM">
+<signal name="SDA_MID/RTC/CAM">
 <contactref element="JP11" pad="9"/>
 <contactref element="U1" pad="33"/>
@@
 <wire x1="101.6" y1="27.94" x2="101.6" y2="50.8" width="0" layer="19" extent="1-1"/>
 </signal>
-<signal name="NC16">
-<contactref element="JP11" pad="16"/>
-</signal>
-<signal name="NC14">
-<contactref element="JP11" pad="14"/>
-</signal>
 <signal name="RFM_MOSI">
 <contactref element="U4" pad="11P"/>
@@
 <wire x1="7.017996875" y1="5.727559375" x2="2.54" y2="20.575" width="0" layer="19" extent="1-1"/>
 </signal>
-<signal name="IM_RXD">
+<signal name="IM_RX">
 <contactref element="U2" pad="18"/>
 <contactref element="U1" pad="26"/>
 <wire x1="13.037659375" y1="27.7304" x2="47.858" y2="5.984" width="0" layer="19" extent="1-1"/>
 </signal>
-<signal name="IM_TXD">
+<signal name="IM_TX">
 <contactref element="U2" pad="19"/>
 <contactref element="U1" pad="6"/>
