File: projects/NECTEC/LRTU/communication_module_20190805.sch (EAGLE design)
At the start: 47 parts, among them Q1 BC847BS, U1 ESP-WROOM-32U (w/uFL), U2 IMAS980TH, U3 WG209_3E6, U4 RFM95W_SMT, X1 uFL, X2 uFL

Commit message: Update the communication board design, and, make PDFs.
Other:
- note added: "ESP32 features three UARTs: UART0 -- for programming RX: IO3 TX: IO1 UART1 -- for AT-command service RX: IO16 TX: IO17 UART2 -- for eMOD RX: IO34 (input only) TX: IO4"
- note removed: "ESP32 features three UARTs: UART0 -- for programming RX: IO3 TX: IO1 UART1 -- for AT-command service RX: IO16 TX: IO17 UART2 -- for eMOD RX: IO34 TX: IO4"
Changed lines of the file:
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@@
     TX: IO17
 UART2 -- for eMOD
-    RX: IO34
+    RX: IO34 (input only)
     TX: IO4</text>
 </plain>
@@
 </instance>
 <instance part="FRAME1" gate="G$1" x="0" y="0" smashed="yes">
-<attribute name="DRAWING_NAME" x="217.17" y="15.24" size="2.54" layer="94"/>
-<attribute name="LAST_DATE_TIME" x="217.17" y="10.16" size="2.286" layer="94"/>
+<attribute name="DRAWING_NAME" x="217.17" y="15.24" size="1.27" layer="94"/>
+<attribute name="LAST_DATE_TIME" x="217.17" y="10.16" size="1.27" layer="94"/>
 <attribute name="SHEET" x="230.505" y="5.08" size="2.54" layer="94"/>
 </instance>

Commit message: Revise many things after dealing with Aj.Doy.
Connections:
- net IM_RXD renamed IM_RX
- net IM_TXD renamed IM_TX
- net SCL0_MID/RTC/CAM renamed SCL_MID/RTC/CAM
- net SDA0_MID/RTC/CAM renamed SDA_MID/RTC/CAM
- net SPI1_CE0_1U renamed SPI_CE0_1U
- net SPI1_CE1_1U renamed SPI_CE1_1U
- net SPI1_MISO_1U renamed SPI_MISO_1U
- net SPI1_MOSI_1U renamed SPI_MOSI_1U
- net SPI1_SCLK_1U renamed SPI_SCLK_1U
- removed net NC14: JP11.14
- removed net NC16: JP11.16
Other:
- moved on the sheet: LED1, R6
Changed lines of the file:
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@@
 <sheet>
 <plain>
-<text x="167.64" y="116.84" size="1.27" layer="91">ESP32 features three SPIs:
+<text x="45.72" y="106.68" size="1.27" layer="91">ESP32 features three SPIs:
   SPI, HSPI and VSPI,
   in slave and master modes.
@@
     3) Micro SDCard interfacings.</text>
 <text x="217.17" y="20.32" size="2.54" layer="94">Author: iPAS</text>
-<text x="45.72" y="99.06" size="1.27" layer="91">ESP32 features three UARTs:
+<text x="167.64" y="114.3" size="1.27" layer="91">ESP32 features three UARTs:
 UART0 -- for programming
     RX: IO3
@@
 <attribute name="VALUE" x="231.14" y="53.34" size="1.27" layer="96"/>
 </instance>
-<instance part="P+1" gate="1" x="205.74" y="71.12" smashed="yes" rot="R90">
-<attribute name="VALUE" x="201.676" y="70.612" size="1.27" layer="96" rot="MR0"/>
+<instance part="P+1" gate="1" x="210.82" y="71.12" smashed="yes" rot="R90">
+<attribute name="VALUE" x="206.756" y="70.612" size="1.27" layer="96" rot="MR0"/>
 </instance>
 <instance part="U1" gate="G$1" x="109.22" y="134.62" smashed="yes">
@@
 <attribute name="VALUE" x="17.78" y="144.78" size="1.778" layer="96"/>
 </instance>
-<instance part="LED1" gate="G$1" x="154.94" y="119.38" smashed="yes">
-<attribute name="NAME" x="155.448" y="115.824" size="1.778" layer="95"/>
-<attribute name="VALUE" x="155.448" y="113.665" size="1.778" layer="96"/>
-</instance>
-<instance part="SUPPLY14" gate="GND" x="154.94" y="111.76" smashed="yes" rot="MR0">
-<attribute name="VALUE" x="154.94" y="109.22" size="1.778" layer="96" rot="MR0"/>
+<instance part="LED1" gate="G$1" x="154.94" y="121.92" smashed="yes">
+<attribute name="NAME" x="155.448" y="118.364" size="1.778" layer="95"/>
+<attribute name="VALUE" x="155.448" y="116.205" size="1.778" layer="96"/>
+</instance>
+<instance part="SUPPLY14" gate="GND" x="154.94" y="114.3" smashed="yes" rot="MR0">
+<attribute name="VALUE" x="154.94" y="111.76" size="1.778" layer="96" rot="MR0"/>
 </instance>
 <instance part="U2" gate="G$1" x="119.38" y="71.12" smashed="yes">
@@
 <attribute name="VALUE" x="198.12" y="24.13" size="1.778" layer="96"/>
 </instance>
-<instance part="R6" gate="G$1" x="149.86" y="121.92" smashed="yes" rot="MR180">
-<attribute name="NAME" x="146.05" y="123.4186" size="1.778" layer="95"/>
-<attribute name="VALUE" x="146.05" y="120.142" size="1.778" layer="96" rot="MR180"/>
+<instance part="R6" gate="G$1" x="149.86" y="124.46" smashed="yes" rot="MR180">
+<attribute name="NAME" x="146.05" y="125.9586" size="1.778" layer="95"/>
+<attribute name="VALUE" x="146.05" y="122.682" size="1.778" layer="96" rot="MR180"/>
 </instance>
 <instance part="JP5" gate="G$1" x="35.56" y="30.48" smashed="yes" rot="R90">
@@
 </busses>
 <nets>
-<net name="SPI1_MISO_1U" class="0">
+<net name="SPI_MISO_1U" class="0">
 <segment>
 <pinref part="JP11" gate="A" pin="4"/>
@@
 </segment>
 </net>
-<net name="SPI1_MOSI_1U" class="0">
+<net name="SPI_MOSI_1U" class="0">
 <segment>
 <pinref part="JP11" gate="A" pin="6"/>
@@
 </segment>
 </net>
-<net name="SPI1_CE1_1U" class="0">
+<net name="SPI_CE1_1U" class="0">
 <segment>
 <pinref part="JP11" gate="A" pin="12"/>
@@
 </segment>
 </net>
-<net name="SPI1_CE0_1U" class="0">
+<net name="SPI_CE0_1U" class="0">
 <segment>
 <pinref part="JP11" gate="A" pin="10"/>
@@
 </segment>
 </net>
-<net name="SPI1_SCLK_1U" class="0">
+<net name="SPI_SCLK_1U" class="0">
 <segment>
 <pinref part="JP11" gate="A" pin="8"/>
@@
 </segment>
 </net>
-<net name="SCL0_MID/RTC/CAM" class="0">
+<net name="SCL_MID/RTC/CAM" class="0">
 <segment>
 <pinref part="JP11" gate="A" pin="7"/>
@@
 </segment>
 </net>
-<net name="SDA0_MID/RTC/CAM" class="0">
+<net name="SDA_MID/RTC/CAM" class="0">
 <segment>
 <pinref part="JP11" gate="A" pin="9"/>
@@
 <pinref part="JP11" gate="A" pin="23"/>
 <pinref part="P+1" gate="1" pin="+5V"/>
-<wire x1="215.9" y1="71.12" x2="205.74" y2="71.12" width="0.1524" layer="91"/>
+<wire x1="215.9" y1="71.12" x2="210.82" y2="71.12" width="0.1524" layer="91"/>
 </segment>
 </net>
@@
 </segment>
 </net>
-<net name="NC16" class="0">
-<segment>
-<pinref part="JP11" gate="A" pin="16"/>
-<wire x1="223.52" y1="81.28" x2="231.14" y2="81.28" width="0.1524" layer="91"/>
-<label x="231.14" y="81.28" size="1.27" layer="95" xref="yes"/>
-</segment>
-</net>
-<net name="NC14" class="0">
-<segment>
-<pinref part="JP11" gate="A" pin="14"/>
-<wire x1="223.52" y1="83.82" x2="231.14" y2="83.82" width="0.1524" layer="91"/>
-<label x="231.14" y="83.82" size="1.27" layer="95" xref="yes"/>
-</segment>
-</net>
 <net name="RFM_MOSI" class="0">
 <segment>
@@
 </segment>
 </net>
-<net name="IM_RXD" class="0">
+<net name="IM_RX" class="0">
 <segment>
 <pinref part="U2" gate="G$1" pin="RXD"/>
@@
 </segment>
 </net>
-<net name="IM_TXD" class="0">
+<net name="IM_TX" class="0">
 <segment>
 <pinref part="U2" gate="G$1" pin="TXD"/>
@@
 <pinref part="U1" gate="G$1" pin="IO2"/>
 <pinref part="R6" gate="G$1" pin="1"/>
-<wire x1="127" y1="121.92" x2="144.78" y2="121.92" width="0.1524" layer="91"/>
-<label x="129.54" y="122.174" size="1.778" layer="95"/>
-</segment>
-</net>
+<wire x1="127" y1="121.92" x2="127" y2="124.46" width="0.1524" layer="91"/>
+<wire x1="127" y1="124.46" x2="144.78" y2="124.46" width="0.1524" layer="91"/>
+<label x="129.54" y="124.714" size="1.778" layer="95"/>
+</segment>
+</net>
