File: projects/NECTEC/LRTU/communication_module_20190916_bus-revised.brd (EAGLE design)
At the start: 121.1 x 70.6 mm, 43 parts, among them IC1 24LC128ST, J2 MICRO-SD_CARD_SOCKETTINY, Q1 BC847BS, U1 ESP-WROOM-32U (w/uFL), U2 IMAS980TH, U3 WG209_3E6, X1 uFL

Commit message: Revise many things after dealing with Aj.Doy.
Parts:
- removed C6: 100nF, ipas:RCL_C1206
- removed IC1: 24LC128ST, microchip:TSSOP8
- removed J2: MICRO-SD_CARD_SOCKETTINY, SparkFun-Connectors:MICROSD_TINY
- removed TP1, TP2, TP3: TPB1,27, ipas:B1,27
- added J1: MICROSD-9P, OPL_Connector:MICRO-SD9+4P-SMD-16.1X14.5X1.85MM
Connections:
- removed net ADC1_0: TP1.TP, U1.4
- removed net ADC1_3: TP2.TP, U1.5
- removed net DAC1: TP3.TP, U1.10
- removed net N$10: IC1.5
- removed net N$11: IC1.6
- removed net N$12: IC1.3
- removed net N$15: IC1.2
- removed net N$17: IC1.1
- removed net PRTCTL1: JP11.21
- removed net SCL_IO_EXP: JP11.24
- removed net SDA_IO_EXP: JP11.26
- removed net SPI_CE1_1U: JP11.12
- removed net USB_1N: JP11.17
- removed net USB_1P: JP11.19
- new net ESP_SD_CD: J1.9, U1.4
- net +3V3: now also J1.4; no longer C6.1, IC1.8, J2.4
- net +5V: no longer JP11.23
- net GND: now also J1.6, J1.G1, J1.G2, J1.G3, J1.G4; no longer C6.2, IC1.4, IC1.7, J2.6, J2.GND1, J2.GND2, J2.GND3, J2.GND4, J2.GND5, J2.GND6, JP11.22, JP11.30, JP11.32
- net N$7: now also J1.1; no longer J2.9
- net N$8: now also J1.8; no longer J2.1, J2.8
- net RXD_TTL0: now also JP11.25; no longer JP11.20
- net SPI_CE0_1U: now also J1.2; no longer J2.2
- net SPI_MISO_1U: now also J1.7; no longer J2.7
- net SPI_MOSI_1U: now also J1.3; no longer J2.3
- net SPI_SCLK_1U: now also J1.5; no longer J2.5
- net TXD_TTL0: now also JP11.23; no longer JP11.18
- net USB_WN: now also JP11.21; no longer JP11.13
- net USB_WP: now also JP11.22; no longer JP11.15
