File: projects/NECTEC/LRTU/communication_module_20190916_bus-revised.sch (EAGLE design)
At the start: 43 parts, among them IC1 24LC128ST, J2 MICRO-SD_CARD_SOCKETTINY, Q1 BC847BS, U1 ESP-WROOM-32U (w/uFL), U2 IMAS980TH, U3 WG209_3E6, X1 uFL

Commit message: Revise many things after dealing with Aj.Doy.
Parts:
- removed C6: 100nF, ipas:RCL_C-EUC1206
- removed IC1: 24LC128ST, microchip:24LC128ST
- removed J2: MICRO-SD_CARD_SOCKETTINY, SparkFun-Connectors:MICRO-SD_CARD_SOCKETTINY
- removed TP1, TP2, TP3: TPB1,27, ipas:TPB1,27
- added J1: MICROSD-9P, OPL_Connector:MICRO-SD-CARD-HOLDER-9P
Connections:
- removed net ADC1_0: TP1.TP, U1.SENSOR_VP
- removed net ADC1_3: TP2.TP, U1.SENSOR_VN
- removed net DAC1: TP3.TP, U1.IO25
- removed net N$10: IC1.SDA
- removed net N$11: IC1.SCL
- removed net N$12: IC1.A2
- removed net N$15: IC1.A1
- removed net N$17: IC1.A0
- removed net PRTCTL1: JP11.21
- removed net SCL_IO_EXP: JP11.24
- removed net SDA_IO_EXP: JP11.26
- removed net SPI_CE1_1U: JP11.12
- removed net USB_1N: JP11.17
- removed net USB_1P: JP11.19
- new net ESP_SD_CD: J1.CDN, U1.SENSOR_VP
- net +3V3: now also J1.VDD; no longer C6.1, IC1.VCC, J2.VCC
- net +5V: no longer JP11.23
- net GND: now also J1.G1, J1.G2, J1.G3, J1.G4, J1.VSS; no longer C6.2, IC1.GND, IC1.WP, J2.GND, J2.SHIELD, JP11.22, JP11.30, JP11.32
- net N$7: now also J1.DATA2; no longer J2.NC
- net N$8: now also J1.DATA1; no longer J2.RSV
- net RXD_TTL0: now also JP11.25; no longer JP11.20
- net SPI_CE0_1U: now also J1.CS; no longer J2.CS
- net SPI_MISO_1U: now also J1.DO; no longer J2.DO
- net SPI_MOSI_1U: now also J1.DI; no longer J2.DI
- net SPI_SCLK_1U: now also J1.SCLK; no longer J2.SCK
- net TXD_TTL0: now also JP11.23; no longer JP11.18
- net USB_WN: now also JP11.21; no longer JP11.13
- net USB_WP: now also JP11.22; no longer JP11.15
Other:
- moved on the sheet: JP11, SJ1, SJ2, SJ4, SJ5, SJ6, SJ7
