File: projects/NECTEC/NICT2019/esp32_part_20190819.brd (EAGLE design)
At the start: 100 x 80 mm, 51 parts, among them J2 MICRO-SD_CARD_SOCKETTINY, Q1 BC847BS, U1 ESP-WROOM-32U (w/uFL), U2 BME280, U4 RFM95W_SMT, X2 uFL

Commit message: Complete the CM3-ESP32 board roughly.
Parts:
- removed C18: 4.7uF, rcl:C1608
- removed R16, R17: 100K, rcl:R0603
- added C11: 4.7uF, ipas:RCL_150CLZ-1014
- added SJ6: (no value), ipas:SOLDERJUMPER_REFLOW
- added TP_RTC_32K1, TP_RTC_INT1: TPB1,27, ipas:B1,27
- R14, R15: value 100K -> 10k; device rcl:R0603 -> ipas:RCL_M0805
- moved R15 36.1 mm to (-91.4, -280.7)
- moved R14 35.9 mm to (-96.5, -280.7)
Connections:
- net VCC_5V renamed +5V
- removed net CM_VDAC: SODIMM.189, SODIMM.190
- removed net GPIO5: SODIMM.17
- removed net GPIO6: SODIMM.21
- removed net N$10: R14.2, SODIMM.30
- removed net N$11: R17.2, SODIMM.82
- removed net N$8: R16.2, SODIMM.84
- removed net N$9: R15.2, SODIMM.28
- removed net SDX_CLK: SODIMM.10
- removed net SDX_CMD: SODIMM.12
- removed net SDX_D0: SODIMM.16
- removed net SDX_D1: SODIMM.18
- removed net SDX_D2: SODIMM.22
- removed net SDX_D3: SODIMM.24
- removed net TV_DAC: SODIMM.166
- removed net VCC_1V8: SODIMM.183, SODIMM.184, SODIMM.185, SODIMM.186
- removed net VCC_3V3: C18.1, SODIMM.191, SODIMM.192, SODIMM.193, SODIMM.194, SODIMM.39, SODIMM.4, SODIMM.40, SODIMM.41, SODIMM.42, SODIMM.6
- new net CM_CAM0_IO0: SODIMM.36
- new net CM_CAM0_IO1: SODIMM.34
- new net CM_CAM1_IO0: SODIMM.11
- new net CM_CAM1_IO1: SODIMM.9
- net +3V3: now also C11.+, R14.2, R15.2, SODIMM.183, SODIMM.184, SODIMM.185, SODIMM.186, SODIMM.189, SODIMM.190, SODIMM.191, SODIMM.192, SODIMM.193, SODIMM.194, SODIMM.39, SODIMM.4, SODIMM.40, SODIMM.41, SODIMM.42, SODIMM.6
- net CM_SCL0: now also SODIMM.30; no longer SODIMM.5
- net CM_SCL1: now also SODIMM.5; no longer SODIMM.11
- net CM_SDA0: now also SODIMM.28; no longer SODIMM.3
- net CM_SDA1: now also SODIMM.3; no longer SODIMM.9
- net GND: now also C11.-; no longer C18.2, R14.1, R15.1, R16.1, R17.1
